File: learn/pcb/magfire/magfire.kicad_pcb (KiCad board)
At the start: 2 copper layers, 16.5 x 19.5 mm, 3 parts, among them J1 Conn_01x07_Pin, J2 Conn_01x07_Pin, U1 74HC14

Commit message: add image and update BOM
Parts:
- removed J1, J2: Conn_01x07_Pin, Connector_PinHeader_2.54mm:PinHeader_1x07_P2.54mm_Vertical
- removed U1: 74HC14, Package_SO:TSSOP-14_4.4x5mm_P0.65mm
Routing:
- net Net-(J2-Pin_7): track 7.54 -> 0.00 mm
- net Net-(J1-Pin_7): track 7.29 -> 0.00 mm
- net Net-(J1-Pin_1): track 6.95 -> 0.00 mm
- net Net-(J2-Pin_1): track 6.52 -> 0.00 mm
- net Net-(J2-Pin_6): track 6.08 -> 0.00 mm
- net Net-(J1-Pin_6): track 5.83 -> 0.00 mm
- net Net-(J1-Pin_2): track 5.49 -> 0.00 mm
- net Net-(J2-Pin_2): track 5.06 -> 0.00 mm
- net Net-(J1-Pin_5): track 4.35 -> 0.00 mm
- net Net-(J2-Pin_5): track 4.27 -> 0.00 mm
- net Net-(J1-Pin_3): track 4.21 -> 0.00 mm
- net Net-(J2-Pin_3): track 3.85 -> 0.00 mm
- net Net-(J1-Pin_4): track 3.57 -> 0.00 mm
- net Net-(J2-Pin_4): track 3.49 -> 0.00 mm
Other:
- board outline removed
